File: HW/SERVO_POWER_INJECTOR.kicad_pcb (KiCad board)
At the start: 4 copper layers, 28 x 11 mm, 14 parts, among them J1 Conn_01x04, J4 Conn_01x03, U1 AZ1084CD-ADJ

Commit message: WIP Commit
Parts:
- removed 100nF1, 100nF2, 10uF1, 10uF2, 10uF3: C_0603, C_Capacitor:C_0603
- removed 1K1, 1K2, 3K1, 3K2: R_0603, R_Resistor:R_0603
- removed J1: Conn_01x04, Connector_PinHeader_2.54mm:PinHeader_1x04_P2.54mm_Vertical
- removed J4: Conn_01x03, Connector_PinHeader_2.54mm:PinHeader_1x03_P2.54mm_Vertical
- added C1: 10uF 50V, C_Capacitor:C_1206, F.Cu at (206.0, 153.5)
- added C2: 100nF 50V, C_Capacitor:C_0402, F.Cu at (209.2, 150.6)
- added C3: 100nF 50V, C_Capacitor:C_0402, F.Cu at (209.0, 158.7)
- added C4: 1uF 10V, C_Capacitor:C_0402, F.Cu at (208.0, 158.7)
- added C5: 22uF 10V, C_Capacitor:C_0603, F.Cu at (206.8, 158.2)
- added N1: Finger_2.5x4_M1, N_NonPart:Finger_2.5x4_M1, F.Cu at (202.0, 151.2)
- added N2: Finger_2.5x4_M1, N_NonPart:Finger_2.5x4_M1, F.Cu at (202.0, 155.0)
- added N4: Finger_2.5x4_M1, N_NonPart:Finger_2.5x4_M1, F.Cu at (202.0, 158.8)
- added N5: Finger_2.5x4_M1, N_NonPart:Finger_2.5x4_M1, F.Cu at (217.5, 158.8)
- added N6: Finger_2.5x4_M1, N_NonPart:Finger_2.5x4_M1, F.Cu at (217.5, 155.0)
- added N7: Finger_2.5x4_M1, N_NonPart:Finger_2.5x4_M1, F.Cu at (217.5, 151.2)
- added R1: 1K, R_Resistor:R_0402, F.Cu at (214.0, 158.7)
- added R2: 243R 1%, R_Resistor:R_0402, F.Cu at (211.5, 150.6)
- added R3: 732 1%, R_Resistor:R_0402, F.Cu at (213.8, 150.6)
- added R4: 3K 1%, R_Resistor:R_0402, F.Cu at (206.0, 156.3)
- DS1: value DS_0603 -> Red
- U1: value AZ1084CD-ADJ -> LM317EMPX/NOPB; footprint U_IC:TO252-2 -> U_IC:SOT223_3
- moved DS1 63.3 mm to (205.2, 158.2), turned to 90 degrees
- moved U1 55.5 mm to (211.5, 155.5), turned to -90 degrees
- moved G*** 54.2 mm to (209.6, 153.2)
Routing:
- net +5V: track 25.7 -> 1.94 mm
- net /S1_IN: track 17.1 -> 0.00 mm, vias 1 -> 0
- net Net-(N4-Pad1): track 0.00 -> 13.5 mm, vias 0 -> 1
- net GND: track 6.94 -> 15.8 mm, vias 37 -> 9
- net VCC: track 7.20 -> 0.00 mm
- net Net-(U1-ADJ): track 3.87 -> 3.22 mm
- added copper zone on F.Cu, net +5V
- added copper zone on F.Cu, net VCC
- removed copper zone on In1.Cu, net GND
- removed copper zone on In2.Cu, net GND
Other:
- board size 28 x 11 mm -> 11.5 x 10 mm
- copper layers 4 -> 2
- board text added: "B+"
- board text added: "G"
- board text added: "S"
- board text added: "SERVO POWER INJECTOR v2.0"
- board text removed: "+"
- board text removed: "-"
- board text removed: "BATT"
- board text removed: "GND"
- board text removed: "SERVO POWER INJECTOR v1.0"
- board text removed: "SIG"
