File: HW/SERVO_POWER_INJECTOR.kicad_sch (KiCad schematic)
At the start: 13 parts, among them J1 Conn_01x04, J4 Conn_01x03, U1 AZ1084CD-ADJ

Commit message: WIP Commit
Parts:
- removed 100nF1, 100nF2, 10uF1, 10uF2, 10uF3: C_0603, C_Capacitor:C_0603, symbol C_Capacitor:C_0603
- removed 1K1, 1K2, 3K1, 3K2: R_0603, R_Resistor:R_0603, symbol R_Resistor:R_0603
- removed J1: Conn_01x04, Connector_PinHeader_2.54mm:PinHeader_1x04_P2.54mm_Vertical, symbol Connector_Generic:Conn_01x04
- removed J4: Conn_01x03, Connector_PinHeader_2.54mm:PinHeader_1x03_P2.54mm_Vertical, symbol Connector_Generic:Conn_01x03
- removed U1: AZ1084CD-ADJ, U_IC:TO252-2, symbol U_Power:AZ1084CD-ADJ
- added C1: 10uF 50V, C_Capacitor:C_1206, symbol C_Capacitor:C_1206
- added C2, C3: 100nF 50V, C_Capacitor:C_0402, symbol C_Capacitor:C_0402
- added C4: 1uF 10V, C_Capacitor:C_0402, symbol C_Capacitor:C_0402
- added C5: 22uF 10V, C_Capacitor:C_0603, symbol C_Capacitor:C_0603
- added N1, N2, N4, N5, N6, N7: Finger_2.5x4_M1, N_NonPart:Finger_2.5x4_M1, symbol N_NonPart:Finger_2.5x4_M1
- added R1: 1K, R_Resistor:R_0402, symbol R_Resistor:R_0402
- added R2: 243R 1%, R_Resistor:R_0402, symbol R_Resistor:R_0402
- added R3: 732 1%, R_Resistor:R_0402, symbol R_Resistor:R_0402
- added R4: 3K 1%, R_Resistor:R_0402, symbol R_Resistor:R_0402
- added U1: LM317EMPX/NOPB, U_IC:SOT223_3, symbol U_Power:LM317EMPX/NOPB
- DS1: value DS_0603 -> Red; LCSC Part (none) -> C965799; MFG Part  (none) -> XL-1608SURC-06
Connections:
- net +5V: now also C3.1, C4.1, C5.1, N6.1, R2.1, R4.1, U1.2 (VOUT)
- net GND: now also C1.2, C2.2, C3.2, C4.2, C5.2, N2.1, N7.1, R3.2
- net S1: now also N5.1, R1.2
- net VCC: now also C1.1, C2.1, N1.1, U1.3 (VIN)
- net at DS1.2 (A): now also R4.2
- new net: R2.2, R3.1, U1.1 (ADJ)
- new net: N4.1, R1.1
